File: hardware/noisy_cricket_sao.kicad_pcb (KiCad board)
At the start: 2 copper layers, 30 x 25 mm, 25 parts, among them J1 SAO 6-Pin, J2 Debug Pogo 6-Pin, U1 AD8107, U2 CH32V003F4U6

Commit message: Initial ugly routing of PCB
Parts:
- added MECH1: 1510-8Ω1W-L60MM_MECH, noisy_cricket_sao:1510-8Ω1W-L60MM_MECH, F.Cu at (142.7, 84.7)
- SPK1: footprint noisy_cricket_sao:1510-8Ω1W-L60MM -> noisy_cricket_sao:1510-8Ω1W-L60MM_SMT_PADS
- moved R5 22.1 mm to (133.3, 80.4), turned to 180 degrees
- moved R6 21.0 mm to (133.3, 81.4), turned to 180 degrees
- moved R7 21.0 mm to (133.3, 82.4), turned to 180 degrees
- moved SPK1 14.2 mm to (129.2, 88.2), turned to 0 degrees
- moved R10 7.32 mm to (146.2, 95.4), turned to 90 degrees
- moved R8 6.94 mm to (148.6, 99.5), turned to 0 degrees
- moved MIC1 6.75 mm to (153.2, 86.3), turned to 0 degrees
- moved J2 6.51 mm to (149.2, 101.7)
- moved R9 6.40 mm to (147.3, 95.4), turned to 90 degrees
- moved C7 6.10 mm to (153.6, 83.9), turned to 0 degrees
- moved U2 3.47 mm to (152.2, 92.0)
- moved C1 2.75 mm to (131.0, 97.8)
- moved C2 2.75 mm to (133.5, 99.3)
- moved C3 2.75 mm to (132.0, 99.8)
- moved C4 2.75 mm to (133.5, 96.3)
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Connections:
- U1 pad 9: (no net) -> GND
- U2 pad 16: /LED_B -> /LED_R
- U2 pad 18: /LED_R -> /LED_B
- U2 pad 21: (no net) -> GND
- U2 pad 3: unconnected-(U2-PA2_OSCO-Pad3) -> /AMP_SD
Routing:
- net +3V3: track 1.36 -> 113.0 mm
- net /AMP_SD: track 0.00 -> 32.9 mm
- net /LED_R: track 0.00 -> 27.0 mm
- net /LED_G: track 0.00 -> 26.7 mm
- net /LED_B: track 0.00 -> 26.2 mm
- net /AUDIO: track 0.00 -> 22.7 mm
- net /RESET: track 0.00 -> 22.5 mm, vias 0 -> 2
- net /UART: track 0.00 -> 16.6 mm, vias 0 -> 2
- net /SCL: track 0.00 -> 16.1 mm
- net /SDA: track 0.00 -> 15.9 mm
- net /SWIO: track 0.00 -> 15.1 mm, vias 0 -> 2
- net Net-(SPK1-+): track 3.66 -> 18.3 mm
- net GND: track 1.36 -> 14.3 mm, vias 0 -> 9
- net /PDM_DATA: track 0.00 -> 8.47 mm
- net /PDM_CLK: track 0.00 -> 7.55 mm
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Other:
- board text added: "2026"
- board text added: "github.com/bmellor/ noisy_cricket_sao"

Commit message: 2nd ugly route complete
Parts:
- removed J2: Debug Pogo 6-Pin, noisy_cricket_sao:Debug Pogo 6-Pin
- removed R10, R9: 10k, Resistor_SMD:R_0402_1005Metric
- added FID1: Fiducial, Fiducial:Fiducial_0.5mm_Mask1.5mm, F.Cu at (129.3, 102.2)
- added FID2: Fiducial, Fiducial:Fiducial_0.5mm_Mask1.5mm, F.Cu at (153.2, 81.1)
- added TP1: TestPoint, TestPoint:TestPoint_Pad_D1.0mm, F.Cu at (131.6, 93.7)
- moved C7 17.3 mm to (151.8, 101.1), turned to -90 degrees
- moved U2 16.8 mm to (135.4, 92.4), turned to 45 degrees
- moved C8 14.9 mm to (135.9, 96.3), turned to 90 degrees
- moved MIC1 14.9 mm to (149.4, 100.7), turned to -90 degrees
- moved R8 13.5 mm to (135.3, 102.0)
Connections:
- J1 pad 5: unconnected-(J1-GPIO1-Pad5) -> /UART
- J1 pad 6: unconnected-(J1-GPIO2-Pad6) -> /SWIO
- U2 pad 19: /UART -> unconnected-(U2-PD5-Pad19)
- U2 pad 20: /UART -> unconnected-(U2-PD6-Pad20)
- U2 pad 7: unconnected-(U2-PC0-Pad7) -> /UART
Routing:
- net +3V3: track 113.0 -> 82.6 mm
- net /SWIO: track 15.1 -> 42.7 mm, vias 2 -> 0
- net /RESET: track 22.5 -> 2.58 mm, vias 2 -> 0
- net /LED_B: track 26.2 -> 9.69 mm
- net /LED_G: track 26.7 -> 10.2 mm
- net /LED_R: track 27.0 -> 11.0 mm
- net /AMP_SD: track 32.9 -> 18.3 mm
- net /AUDIO: track 22.7 -> 8.10 mm
- net /UART: track 16.6 -> 3.43 mm, vias 2 -> 0
- net /PDM_CLK: track 7.55 -> 20.3 mm
- net /PDM_DATA: track 8.47 -> 18.8 mm
- net /SDA: track 15.9 -> 6.64 mm
- net /SCL: track 16.1 -> 12.8 mm
- net GND: track 14.3 -> 14.7 mm, vias 9 -> 7
Other:
- board text added: "RST"

Commit message: cleaned up routing
Parts:
- moved C7 1.50 mm to (150.6, 100.3)
- moved MIC1 1.43 mm to (148.0, 100.7)
- moved FID2 0.64 mm to (152.7, 80.7)
- moved R8 0.53 mm to (135.4, 102.5)
- moved FID1 0.43 mm to (129.6, 102.5)
- moved C8 0.28 mm to (135.9, 96.0), turned to -90 degrees
- moved TP1 0.15 mm to (131.8, 93.7)
Routing:
- net +3V3: track 82.6 -> 76.8 mm
- net /SWIO: track 42.7 -> 37.6 mm
- net /SCL: track 12.8 -> 17.5 mm
- net GND: track 14.7 -> 19.1 mm, vias 7 -> 9
- net /AMP_SD: track 18.3 -> 17.2 mm
- net /SDA: track 6.64 -> 7.33 mm
- net /PDM_DATA: track 18.8 -> 18.2 mm
- added copper zone on F.Cu, net GND
