File: hardware/noisy_cricket_sao.kicad_sch (KiCad schematic)
At the start: 23 parts, among them J1 SAO 6-Pin, U1 AD8107, U3 MSPM0C1104SDYYR

Commit message: Update LPF for 1x gain, tweak footprints and silk
Parts:
- C1: value 220pF -> 820pF
- C7: value 0.39uF -> 1uF
- R2: value 68k -> 20k
Changed lines of the file:
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@@
 			)
 		)
-		(property "Value" "68k"
+		(property "Value" "20k"
 			(at 74.93 48.2599 0)
 			(show_name no)
@@
 			)
 		)
-		(property "Value" "220pF"
+		(property "Value" "820pF"
 			(at 89.408 48.26 0)
 			(show_name no)
@@
 			)
 		)
-		(property "Value" "0.39uF"
+		(property "Value" "1uF"
 			(at 170.18 95.2499 0)
 			(show_name no)
